File: hardware/templogger.kicad_sch (KiCad schematic)
At the start: 49 parts, among them J102 Conn_01x02, J103 USB_B_Mini, J104 LiPo BATTERY, J105 CPROBE, J401 Conn_K_TERM_XH_2P, Q102 IRF7606PBF, Q201 2N7002K, SW101 BOOT, SW101 SW_Push_LED, SW102 RESET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

Commit message: Add gerber file and update BOM list
Parts:
- removed J105: CPROBE, Connector_PinHeader_1.27mm:PinHeader_1x02_P1.27mm_Vertical, symbol tbctl:PinHeader Conn_01x02
- added C101: 0.1uF, Capacitor_SMD:C_0603_1608Metric_Pad1.08x0.95mm_HandSolder, symbol Device:C
- added JP101: SolderJumper_2_Open, Jumper:SolderJumper-2_P1.3mm_Open_RoundedPad1.0x1.5mm, symbol tbctl:SolderJumper_2_Open
- added R101: 10K, tbctl:R_0805_2012Metric_Pad1.20x1.40mm_HandSolder, symbol Device:R
- added SW105: SLIDE_SW IS-1245T-G, tbctl:SLIDE_SW_IS1235-G, symbol tbctl:SLIDE_SW
- C101, C102: digikey (none) -> 311-1751-1-ND; storeURL (none) -> https://www.digikey.com/en/products/detail/yageo/CC0603JRNP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
- C301, C303, C401: digikey (none) -> 311-1824-1-ND; storeURL (none) -> https://www.digikey.com/en/products/detail/yageo/CC0603MRX7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
- C302, C304: digikey (none) -> 311-3494-1-ND; storeURL (none) -> https://www.digikey.com/en/products/detail/yageo/CC0603MRX5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
- C302: digikey (none) -> 311-1455-1-ND; storeURL (none) -> https://www.digikey.com/en/products/detail/yageo/CC0603KRX5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
- C305: digikey (none) -> 13-CC0603KPX7R7BB105CT-ND; storeURL (none) -> https://www.digikey.com/en/products/detail/yageo/CC0603KPX7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
- D105: digikey (none) -> NSR0340HT1GOSCT-ND; storeURL (none) -> https://www.digikey.com/en/products/detail/onsemi/NSR0340HT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
- D302: value LED GREEN -> LED GREEN SML-E12P8WT86; digikey (none) -> 511-1585-1-ND; storeURL (none) -> https://www.digikey.com/en/products/detail/rohm-semiconduct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
- D302: value LED RED -> LED RED SML-E12V8WT86; digikey (none) -> 511-1587-1-ND; storeURL (none) -> https://www.digikey.com/en/products/detail/rohm-semiconduct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
- FB301: digikey (none) -> 240-2399-1-ND; storeURL (none) -> https://www.digikey.com/en/products/detail/laird-signal-int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
- J102: akizuki (none) -> C-12247; digikey (none) -> 455-2247-ND; storeURL (none) -> https://www.digikey.com/en/products/detail/jst-sales-americ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
- J103: akizuki (none) -> C-02235; storeURL (none) -> https://akizukidenshi.com/catalog/g/gC-02235/
- J104: value LiPo BATTERY -> LiPo BATTERY Socket; akizuki (none) -> C-12802; digikey (none) -> 455-1704-ND; storeURL (none) -> https://www.digikey.com/en/products/detail/jst-sales-americ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
- J401: akizuki (none) -> P-14972; digikey (none) -> 1568-1306-ND; storeURL (none) -> https://www.digikey.com/en/products/detail/sparkfun-electro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
- Q102: value IRF7606PBF -> IRF7606TRPBF; digikey (none) -> IRF7606TRPBFCT-ND; storeURL (none) -> https://www.digikey.com/en/products/detail/infineon-technol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
- Q201: digikey (none) -> 2N7002K-7DICT-ND; storeURL (none) -> https://www.digikey.com/en/products/detail/diodes-incorpora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
- R101, R102, R201, R304: digikey (none) -> 13-RC0603JR-1010KLCT-ND; storeURL (none) -> https://www.digikey.com/en/products/detail/yageo/RC0603JR-1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
- R107: digikey (none) -> 311-2.0KGRCT-ND; storeURL (none) -> https://www.digikey.com/en/products/detail/yageo/RC0603JR-0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
- R107: value 0.1 -> 20K 1%; digikey (none) -> 13-RC0603FR-1320KLCT-ND; storeURL (none) -> https://www.digikey.com/en/products/detail/yageo/RC0603FR-1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
- R107: value 10K -> 20K 1%; digikey (none) -> 13-RC0603FR-1320KLCT-ND; storeURL (none) -> https://www.digikey.com/en/products/detail/yageo/RC0603FR-1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
- R202, R305: digikey (none) -> 311-330GRCT-ND; storeURL (none) -> https://www.digikey.com/en/products/detail/yageo/RC0603JR-0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
- R302: digikey (none) -> 13-RC0603FR-1320KLCT-ND; storeURL (none) -> https://www.digikey.com/en/products/detail/yageo/RC0603FR-1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
- R303: digikey (none) -> 311-12.0KHRCT-ND; storeURL (none) -> https://www.digikey.com/en/products/detail/yageo/RC0603FR-0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
- R304: digikey (none) -> 311-100KGRCT-ND; storeURL (none) -> https://www.digikey.com/en/products/detail/yageo/RC0603JR-0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
- SW101: akizuki (none) -> P-13871; storeURL (none) -> https://akizukidenshi.com/catalog/g/gP-13871/
- SW101: value BOOT -> BOOT TS-06104; akizuki (none) -> P-15969; storeURL (none) -> https://akizukidenshi.com/catalog/g/gP-15969/
- SW102: value RESET -> RESET TS-06104; akizuki (none) -> P-15969; storeURL (none) -> https://akizukidenshi.com/catalog/g/gP-15969/
- SW102: akizuki (none) -> P-13870; storeURL (none) -> https://akizukidenshi.com/catalog/g/gP-13870/
- U101: akizuki (none) -> M-17493; digikey (none) -> 1965-ESP32-C3-WROOM-02-N4CT-ND; storeURL (none) -> https://www.digikey.com/en/products/detail/espressif-system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
- U101: akizuki (none) -> I-13288; digikey (none) -> MCP73831T-2ACI/OTCT-ND; storeURL (none) -> https://www.digikey.com/en/products/detail/microchip-techno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
- U202: storeURL (none) -> https://www.amazon.co.jp/gp/product/B08CTZVVLS/
- U301: digikey (none) -> 1016-1871-1-ND; storeURL (none) -> https://www.digikey.com/en/products/detail/maxlinear-inc/SP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
- U401: akizuki (none) -> I-14486; digikey (none) -> MAX31855KASA+TCT-ND; storeURL (none) -> https://www.digikey.com/en/products/detail/analog-devices-i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
- Y101: storeURL (none) -> https://www.digikey.com/en/products/detail/raltron-electron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
Connections:
- net GND: now also R107.2, C101.2, R101.2; no longer J103.6 (Shield)
- net GPIO2: now also R107.1
- net at FB301.2: now also JP101.1 (A), SW105.2 (B); no longer R107.1
- net at C301.1, C302.1, U301.1 (IN)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: now also JP101.2 (B), SW105.1 (A); no longer R107.2
- new net: C101.1, J103.6 (Shield), R101.1
- no-connect marks 1 -> 2
Other:
- moved on the sheet: FB301, J103

Commit message: Fixed battery socket
Connections:
- net +3.3V: no longer R107.1
- net GND: now also J104.1 (Pin_1); no longer J104.2 (Pin_2)
- net VBAT: now also J104.2 (Pin_2); no longer J104.1 (Pin_1)
- net VIN: now reaches C301.1, C302.1, JP101.2 (B), SW105.1 (A), U301.1 (IN), U301.3 (EN)
- net VIN: now also R107.1
Changed lines of the file:
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@@
   (title_block
     (title "TempLogger")
-    (date "2023-05-02")
-    (rev "Rev2")
+    (date "2023-08-24")
+    (rev "Rev4")
     (company "HNZ")
     (comment 1 "Licensed under CC-BY-SA V4.0")
@@
     (stroke (width 0) (type default))
   )
-  (wire (pts (xy 187.96 114.3) (xy 201.93 114.3))
-    (stroke (width 0) (type default))
-  )
   (wire (pts (xy 96.52 27.94) (xy 110.49 27.94))
     (stroke (width 0) (type default))
@@
     (stroke (width 0) (type default))
   )
-  (wire (pts (xy 199.39 116.84) (xy 199.39 120.65))
+  (wire (pts (xy 199.39 114.3) (xy 199.39 120.65))
     (stroke (width 0) (type default))
   )
@@
     (stroke (width 0) (type default))
   )
+  (wire (pts (xy 154.94 120.65) (xy 166.37 120.65))
+    (stroke (width 0) (type default))
+  )
   (wire (pts (xy 67.31 119.38) (xy 91.44 119.38))
     (stroke (width 0) (type default))
@@
     (stroke (width 0) (type default))
   )
+  (wire (pts (xy 201.93 114.3) (xy 199.39 114.3))
+    (stroke (width 0) (type default))
+  )
   (wire (pts (xy 248.92 66.04) (xy 240.03 66.04))
     (stroke (width 0) (type default))
@@
     (stroke (width 0) (type default))
   )
-  (wire (pts (xy 201.93 116.84) (xy 199.39 116.84))
+  (wire (pts (xy 184.15 116.84) (xy 201.93 116.84))
     (stroke (width 0) (type default))
   )
@@
     (effects (font (size 1.27 1.27)) (justify right bottom))
   )
+  (label "VIN" (at 166.37 120.65 180) (fields_autoplaced)
+    (effects (font (size 1.27 1.27)) (justify right bottom))
+  )
+  (label "VIN" (at 77.47 21.59 180) (fields_autoplaced)
+    (effects (font (size 1.27 1.27)) (justify right bottom))
+  )
   (label "GPIO5{slash}TDI" (at 67.31 121.92 0) (fields_autoplaced)
     (effects (font (size 1.27 1.27)) (justify left bottom))
   )
-  (label "VBAT" (at 187.96 114.3 0) (fields_autoplaced)
+  (label "VBAT" (at 184.15 116.84 0) (fields_autoplaced)
     (effects (font (size 1.27 1.27)) (justify left bottom))
   )
@@
         )
       )
-    )
-  )
-  (symbol (lib_id "power:+3.3V") (at 154.94 120.65 0) (unit 1)
-    (in_bom yes) (on_board yes) (dnp no) (fields_autoplaced)
-    (property "Reference" "#PWR0107" (at 154.94 124.46 0)
-      (effects (font (size 1.27 1.27)) hide)
-    )
-    (property "Value" "+3.3V" (at 154.94 115.57 0)
-      (effects (font (size 1.27 1.27)))
-    )
-    (property "Footprint" "" (at 154.94 120.65 0)
-      (effects (font (size 1.27 1.27)) hide)
-    )
-    (property "Datasheet" "" (at 154.94 120.65 0)
-      (effects (font (size 1.27 1.27)) hide)
-    )
-    (pin "1")
-    (instances
-      (project "ESP32C3"
-        (path "/009eae78-518f-491b-bf83-ac6dccccbbfb"
-          (reference "#PWR0107") (unit 1)
-        )
-      )
-      (project "heatpanelcontroller"
-        (path "/58e88479-720b-4b9e-82a0-586074a9c30b/556e5cf8-d98c-4c3b-9c75-5c1844f1715f"
-          (reference "#PWR0208") (unit 1)
-        )
-      )
-      (project "templogger"
-        (path "/792d1191-f80c-48d2-950c-0713cdccb9e7"
-          (reference "#PWR0124") (unit 1)
-        )
-      )
